File: PCB/Test BMP/Test BMP.kicad_pcb (KiCad board)
At the start: 2 copper layers, 5 parts, among them J1 4 pins socket, J2 4 pins socket, U1 BMP581

Commit message: nouvelle ancre pas fini
Other:
- board outline added: 14 x 8 mm
