File: PCB/Hub/HUB2.kicad_pcb (KiCad board)
At the start: 2 copper layers, 98.8 x 85.2 mm, 30 parts, among them IC1 ESP32-DEVKITC-VE, IC2 TCAN1051VDRQ1, J1 B4B-PH-SM4-TB, K1 DSY2Y-S-205H, Q2 2N2220, U1 BMP581, U10 DB301V-5.0-2P, U3 DB301V-5.0-2P, U4 DB301V-5.0-2P, U5 BMI088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

Commit message: Ouvrier_v4_test_DRC
Parts:
- added C4: 100nF, Capacitor_SMD:C_0402_1005Metric_Pad0.74x0.62mm_HandSolder, F.Cu at (137.6, 51.2)
Routing:
- net GNDREF: track 90.2 -> 93.0 mm
- net +3.3V: track 121.6 -> 124.2 mm
Changed lines of the file:
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@@
 		(sheetname "/")
 		(sheetfile "HUB2.kicad_sch")
+		(units
+			(unit
+				(name "A")
+				(pins "1" "2" "3" "4" "8" "7" "6" "5")
+			)
+		)
 		(attr smd)
 		(duplicate_pad_numbers_are_jumpers no)
@@
 		)
 	)
+	(footprint "Capacitor_SMD:C_0402_1005Metric_Pad0.74x0.62mm_HandSolder"
+		(layer "F.Cu")
+		(at 137.5675 51.25)
+		(descr "Capacitor SMD 0402 (1005 Metric), square (rectangular) end terminal, IPC-7351 nominal with elongated pad for handsoldering. (Body size source: IPC-SM-782 page 76, https://www.pcb-3d.com/wordpress/wp-content/uploads/ipc-sm-782a_amendment_1_and_2.pdf)")
+		(tags "capacitor handsolder")
+		(property "Reference" "C4"
+			(at 0 -1.16 0)
+			(layer "F.SilkS")
+			(effects
+				(font
+					(size 1 1)
+					(thickness 0.15)
+				)
+			)
+		)
+		(property "Value" "100nF"
+			(at 3.9325 0 0)
+			(layer "F.Fab")
+			(effects
+				(font
+					(size 1 1)
+					(thickness 0.15)
+				)
+			)
+		)
+		(property "Datasheet" ""
+			(at 0 0 0)
+			(layer "F.Fab")
+			(hide yes)
+			(effects
+				(font
+					(size 1.27 1.27)
+				)
+			)
+		)
+		(property "Description" "Unpolarized capacitor"
+			(at 0 0 0)
+			(layer "F.Fab")
+			(hide yes)
+			(effects
+				(font
+					(size 1.27 1.27)
+				)
+			)
+		)
+		(property "KiLib_Generator" "SMD_2terminal_chip_molded"
+			(at 0 0 0)
+			(layer "F.SilkS")
+			(hide yes)
+			(effects
+				(font
+					(size 1 1)
+					(thickness 0.15)
+				)
+			)
+		)
+		(property ki_fp_filters "C_*")
+		(sheetname "/")
+		(sheetfile "HUB2.kicad_sch")
+		(units
+			(unit
+				(name "A")
+				(pins "1" "2")
+			)
+		)
+		(attr smd)
+		(duplicate_pad_numbers_are_jumpers no)
+		(fp_line
+			(start -0.115835 -0.36)
+			(end 0.115835 -0.36)
+			(stroke
+				(width 0.12)
+				(type solid)
+			)
+			(layer "F.SilkS")
+		)
+		(fp_line
+			(start -0.115835 0.36)
+			(end 0.115835 0.36)
+			(stroke
+				(width 0.12)
+				(type solid)
+			)
+			(layer "F.SilkS")
+		)
+		(fp_rect
+			(start -1.09 -0.46)
+			(end 1.09 0.46)
+			(stroke
+				(width 0.05)
+				(type solid)
+			)
+			(fill no)
+			(layer "F.CrtYd")
+		)
+		(fp_rect
+			(start -0.5 -0.25)
+			(end 0.5 0.25)
+			(stroke
+				(width 0.1)
+				(type solid)
+			)
+			(fill no)
+			(layer "F.Fab")
+		)
+		(fp_text user "${REFERENCE}"
+			(at 0 0 0)
+			(layer "F.Fab")
+			(effects
+				(font
+					(size 0.25 0.25)
+					(thickness 0.04)
+				)
+			)
+		)
+		(pad "1" smd roundrect
+			(at -0.5675 0)
+			(size 0.735 0.62)
+			(layers "F.Cu" "F.Mask" "F.Paste")
+			(roundrect_rratio 0.25)
+			(net "+3.3V")
+			(pintype "passive")
+		)
+		(pad "2" smd roundrect
+			(at 0.5675 0)
+			(size 0.735 0.62)
+			(layers "F.Cu" "F.Mask" "F.Paste")
+			(roundrect_rratio 0.25)
+			(net "GNDREF")
+			(pintype "passive")
+		)
+		(embedded_fonts no)
+		(model "${KICAD10_3DMODEL_DIR}/Capacitor_SMD.3dshapes/C_0402_1005Metric.step"
+			(offset
+				(xyz 0 0 0)
+			)
+			(scale
+				(xyz 1 1 1)
+			)
+			(rotate
+				(xyz 0 0 0)
+			)
+		)
+	)
 	(footprint "MountingHole:MountingHole_3.2mm_M3"
 		(layer "F.Cu")
@@
 		(sheetname "/")
 		(sheetfile "HUB2.kicad_sch")
+		(units
+			(unit
+				(name "A")
+				(pins "1" "2" "3" "4" "SH1" "SH2")
+			)
+		)
 		(attr smd)
 		(duplicate_pad_numbers_are_jumpers no)
@@
 	)
 	(segment
+		(start 138.75 51.25)
+		(end 138.135 51.25)
+		(width 0.8)
+		(layer "F.Cu")
+		(net "GNDREF")
+	)
+	(segment
 		(start 155.75 53.75)
 		(end 155.5 54)
@@
 	)
 	(segment
+		(start 139 53.25)
+		(end 139 51.5)
+		(width 0.8)
+		(layer "F.Cu")
+		(net "GNDREF")
+	)
+	(segment
 		(start 146.125 97.75)
 		(end 153.5 97.75)
@@
 	)
 	(segment
+		(start 139 51.5)
+		(end 138.75 51.25)
+		(width 0.8)
+		(layer "F.Cu")
+		(net "GNDREF")
+	)
+	(segment
 		(start 133.365 60.885)
 		(end 133.25 61)
@@
 	)
 	(segment
+		(start 136.155 51.25)
+		(end 137 51.25)
+		(width 1)
+		(layer "F.Cu")
+		(net "+3.3V")
+	)
+	(segment
+		(start 135.905 50.595)
+		(end 136.5 50)
+		(width 1)
+		(layer "F.Cu")
+		(net "+3.3V")
+	)
+	(segment
 		(start 154.5 54.75)
 		(end 152.25 52.5)
@@
 	)
 	(segment
-		(start 136.5 51)
-		(end 150.75 51)
+		(start 149.75 50)
+		(end 152.25 52.5)
 		(width 1)
 		(layer "F.Cu")
@@
 	)
 	(segment
-		(start 135.905 53.059)
-		(end 135.905 51.595)
-		(width 1)
+		(start 154.25 56.7)
+		(end 154.5 56.45)
+		(width 0.4)
 		(layer "F.Cu")
 		(net "+3.3V")
 	)
 	(segment
-		(start 154.25 56.7)
-		(end 154.5 56.45)
-		(width 0.4)
+		(start 135.905 53.059)
+		(end 135.905 51.5)
+		(width 1)
 		(layer "F.Cu")
 		(net "+3.3V")
@@
 	)
 	(segment
+		(start 135.905 51.5)
+		(end 136.155 51.25)
+		(width 1)
+		(layer "F.Cu")
+		(net "+3.3V")
+	)
+	(segment
 		(start 173.5 65.54)
 		(end 173.5 94)
@@
 	)
 	(segment
-		(start 135.905 51.595)
-		(end 136.5 51)
-		(width 1)
-		(layer "F.Cu")
-		(net "+3.3V")
-	)
-	(segment
 		(start 173.25 64.25)
 		(end 172.73 64.77)
@@
 	)
 	(segment
+		(start 135.905 51.5)
+		(end 135.905 50.595)
+		(width 1)
+		(layer "F.Cu")
+		(net "+3.3V")
+	)
+	(segment
 		(start 151.75 95.3)
 		(end 146 95.3)
@@
 	)
 	(segment
+		(start 136.5 50)
+		(end 149.75 50)
+		(width 1)
+		(layer "F.Cu")
+		(net "+3.3V")
+	)
+	(segment
 		(start 155 52.5)
 		(end 158.5 49)
@@
 		(width 1)
 		(layer "F.Cu")
-		(net "+3.3V")
-	)
-	(segment
-		(start 150.75 51)
-		(end 152.25 52.5)
-		(width 1)
-		(layer "F.Cu")
