File: PCB/Hub/Hub.kicad_sch (KiCad schematic)
At the start: 27 parts, among them IC1 ESP32-DEVKITC-VE, IC2 Tranceiver_CAN, J1 Connecteur_male_Grove_Mabee, K1 DSY2Y-S-205H, Q2 2N2222, U1 BMP581, U10 Bornier_a_vis, U3 Bornier_a_vis, U4 DB301V-5.0-2P, U5 BMI088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

Commit message: MaJ Hub nouvelle version relais-bouton-alim
Parts:
- added D2, D3: FR107, Bibliotheque_Projet:Diode FR107, symbol Bibliotheque_Projet:Diode_FR107
- added Q1: 2N2222B, Bibliotheque_Projet:2N2222B, symbol Bibliotheque_Projet:2N2222B
- added R7: 1K, Resistor_THT:R_Axial_DIN0207_L6.3mm_D2.5mm_P10.16mm_Horizontal, symbol Device:R
- D1: value 1N914 -> FR107; footprint Diode_THT:D_DO-41_SOD81_P12.70mm_Horizontal -> Bibliotheque_Projet:Diode FR107; symbol Diode:1N914 -> Bibliotheque_Projet:Diode_FR107
- K1: value DSY2Y-S-205H -> Relais DSY2Y-S-205H
- R4: value 22k -> 10K
- R6: value 8.2k -> 3.3K
Connections:
- net 12V is gone; now on net +12V: K1.13 (COM_2), K1.4 (COM_1), U10.2, U3.2
- net +12V: no longer K1.8 (NO_1), K1.9 (NO_2), U8.1 (12V)
- net +5V: now also K1.1 (COIL_1), D3.1 (K)
- net GNDREF: now also R2.2, R6.1, Q1.1 (E); no longer K1.16 (COIL_2), R6.2, U7.2
- net at IC1.10 (IO26): now also U5.6 (CSB1/NC)
- net at IC1.13 (IO12): now also U7.1
- net at IC1.16 (D2): now also R7.1
- net at IC1.24 (IO2): no longer R2.2
- net at IC1.29 (IO5): no longer U5.6 (CSB1/NC)
- net at IC1.34 (RX): no longer IC2.4 (RXD)
- net at IC1.35 (TX): no longer IC2.1 (TXD)
- net at IC1.6 (IO35): now also R4.2, R6.2; no longer K1.1 (COIL_1)
- net at R4.1, U6.2: now also D2.2 (A); no longer K1.11 (NC_2), K1.6 (NC_1)
- net at R2.1: now also U7.2; no longer U7.1
- new net: D2.1 (K), K1.8 (NO_1), K1.9 (NO_2), U8.1 (12V)
- new net: Q1.2 (B), R7.2
- new net: D3.2 (A), K1.16 (COIL_2), Q1.3 (C)
- now unconnected: IC1.5 (IO34)
Other:
- note added: "Bouton poussoir + LED bouton"
- note added: "Entrée 12V"
- moved on the sheet: D1, LS1, R3, R4, R6, U10, U3, U6, U7
