File: PCB/Hub/Hub.kicad_pcb (KiCad board)
At the start: 2 copper layers, 98.8 x 85.2 mm, 34 parts, among them IC1 ESP32-DEVKITC-VE, IC2 Tranceiver_CAN, J1 Connecteur_male_Grove_Mabee, K1 Relais DSY2Y-S-205H, Q1 2N2222B, Q2 2N2222, U10 Bornier_a_vis, U2 BMP581, U3 Bornier_a_vis, U4 DB301V-5.0-2P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

Commit message: connected INT pins BMI088 KiCad Hub
Connections:
- IC1 pad 3: unconnected-(IC1-VP-Pad3) -> Net-(IC1-VP)
- IC1 pad 4: unconnected-(IC1-VN-Pad4) -> Net-(IC1-VN)
- U5 pad 8: unconnected-(U5-INT1-Pad8) -> Net-(IC1-VN)
- U5 pad 9: unconnected-(U5-INT3-Pad9) -> Net-(IC1-VP)
Changed lines of the file:
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@@
 			(layers "*.Cu" "*.Mask")
 			(remove_unused_layers no)
-			(net "unconnected-(U5-INT1-Pad8)")
+			(net "Net-(IC1-VN)")
 			(pinfunction "INT1_8")
 			(pintype "input")
@@
 			(layers "*.Cu" "*.Mask")
 			(remove_unused_layers no)
-			(net "unconnected-(U5-INT3-Pad9)")
+			(net "Net-(IC1-VP)")
 			(pinfunction "INT3_9")
 			(pintype "input")
@@
 			(layers "*.Cu" "*.Mask")
 			(remove_unused_layers no)
-			(net "unconnected-(IC1-VP-Pad3)")
+			(net "Net-(IC1-VP)")
 			(pinfunction "VP_3")
 			(pintype "passive")
@@
 			(layers "*.Cu" "*.Mask")
 			(remove_unused_layers no)
-			(net "unconnected-(IC1-VN-Pad4)")
+			(net "Net-(IC1-VN)")
 			(pinfunction "VN_4")
 			(pintype "passive")

Commit message: Pin INT BMPA581 connecté KiCad Hub
Connections:
- IC1 pad 29: unconnected-(IC1-IO5-Pad29) -> Net-(IC1-IO5)
- U2 pad 5: unconnected-(U2-INT-Pad5) -> Net-(IC1-IO21)
- U2 pad 6: Net-(IC1-IO21) -> Net-(IC1-IO5)
Changed lines of the file:
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@@
 			(layers "*.Cu" "*.Mask")
 			(remove_unused_layers no)
-			(net "unconnected-(U2-INT-Pad5)")
+			(net "Net-(IC1-IO21)")
 			(pinfunction "INT_5")
 			(pintype "passive")
@@
 			(layers "F.Cu" "F.Mask")
 			(roundrect_rratio 0.1)
-			(net "unconnected-(U2-INT-Pad5)")
+			(net "Net-(IC1-IO21)")
 			(pinfunction "INT_5")
 			(pintype "passive")
@@
 			(layers "*.Cu" "*.Mask")
 			(remove_unused_layers no)
-			(net "Net-(IC1-IO21)")
+			(net "Net-(IC1-IO5)")
 			(pinfunction "CSB_6")
 			(pintype "passive")
@@
 			(layers "F.Cu" "F.Mask")
 			(roundrect_rratio 0.1)
-			(net "Net-(IC1-IO21)")
+			(net "Net-(IC1-IO5)")
 			(pinfunction "CSB_6")
 			(pintype "passive")
@@
 			(layers "*.Cu" "*.Mask")
 			(remove_unused_layers no)
-			(net "unconnected-(IC1-IO5-Pad29)")
+			(net "Net-(IC1-IO5)")
 			(pinfunction "IO5_29")
 			(pintype "passive")
