File: PCB/Ouvrier/Ouvrier.kicad_sch (KiCad schematic)
At the start: 8 parts, among them J1 Conn_01x02, Q1 2N2220, U1 XIAO-ESP32-S3-Plus-SMD, U2 BMP581, U3 UWB

Commit message: MaJ KiCad ouvrier BMP581
Parts:
- removed J1: Conn_01x02, Bibliotheque_Projet:CONN-TH_2P-P5.00_L7.6-W10.0, symbol Connector_Generic:Conn_01x02
- U1: value XIAO-ESP32-S3-Plus-SMD -> XIAO-ESP32-S3-Plus-DIP
- U2: footprint BMP581 -> Bibliotheque_Projet:BMP581; symbol BMP581:BMP581 -> Bibliotheque_Projet:BMP581
Changed lines of the file:
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@@
-	(wire
-		(pts
-			(xy 140.97 43.18) (xy 128.27 43.18)
-		)
-		(stroke
-			(width 0)
-			(type default)
-		)
-	)
 	(wire
 		(pts
@@
 	(wire
 		(pts
-			(xy 128.27 43.18) (xy 128.27 40.64)
+			(xy 140.97 40.64) (xy 140.97 83.82)
 		)
 		(stroke
@@
 	(wire
 		(pts
-			(xy 128.27 40.64) (xy 224.79 40.64)
+			(xy 140.97 40.64) (xy 224.79 40.64)
 		)
 		(stroke
@@
 		(pts
 			(xy 48.26 71.12) (xy 48.26 146.05)
-		)
-		(stroke
-			(width 0)
-			(type default)
-		)
-	)
-	(wire
-		(pts
-			(xy 140.97 83.82) (xy 140.97 43.18)
 		)
 		(stroke
@@
 	)
 	(symbol
-		(lib_id "BMP581:BMP581")
+		(lib_id "Bibliotheque_Projet:BMP581")
 		(at 49.53 143.51 0)
 		(unit 1)
@@
 			)
 		)
-		(property "Footprint" "BMP581"
+		(property "Footprint" "Bibliotheque_Projet:BMP581"
 			(at 76.2 228.27 0)
 			(hide yes)
@@
 			)
 		)
-		(property "Value" "XIAO-ESP32-S3-Plus-SMD"
+		(property "Value" "XIAO-ESP32-S3-Plus-DIP"
 			(at 160.655 78.74 0)
 			(show_name no)
@@
 					(unit 1)
 				)
-			)
-		)
-	)
-	(symbol
-		(lib_id "Connector_Generic:Conn_01x02")
-		(at 49.53 39.37 0)
-		(unit 1)
-		(body_style 1)
-		(exclude_from_sim no)
-		(in_bom yes)
-		(on_board yes)
-		(in_pos_files yes)
-		(dnp no)
-		(fields_autoplaced yes)
-		(property "Reference" "J1"
-			(at 52.07 39.3699 0)
-			(show_name no)
-			(do_not_autoplace no)
-			(effects
-				(font
-					(size 1.27 1.27)
-				)
-				(justify left)
-			)
-		)
-		(property "Value" "Conn_01x02"
-			(at 52.07 41.9099 0)
-			(show_name no)
-			(do_not_autoplace no)
-			(effects
-				(font
-					(size 1.27 1.27)
-				)
-				(justify left)
-			)
-		)
-		(property "Footprint" "Bibliotheque_Projet:CONN-TH_2P-P5.00_L7.6-W10.0"
-			(at 49.53 39.37 0)
-			(hide yes)
-			(show_name no)
-			(do_not_autoplace no)
-			(effects
-				(font
-					(size 1.27 1.27)
-				)
-			)
-		)
-		(property "Datasheet" ""
-			(at 49.53 39.37 0)
-			(hide yes)
-			(show_name no)
-			(do_not_autoplace no)
-			(effects
-				(font
-					(size 1.27 1.27)
-				)
-			)
-		)
-		(property "Description" "Generic connector, single row, 01x02, script generated (kicad-library-utils/schlib/autogen/connector/)"
-			(at 49.53 39.37 0)
-			(hide yes)
-			(show_name no)
-			(do_not_autoplace no)
-			(effects
-				(font
-					(size 1.27 1.27)
-				)
-			)
-		)
-		(pin "2"
-		)
-		(pin "1"
-		)
-		(instances
-			(project "Ouvrier"
-				(path "/84605c1a-5009-408b-9a0f-13132cab7487"
-					(reference "J1")
-					(unit 1)
-				)

Commit message: MaJ batterie KiCad Ouvrier
Parts:
- removed Q1: 2N2220, Package_TO_SOT_THT:TO-39-3, symbol Transistor_BJT:2N2219
- added Q1: 2N2222B, Bibliotheque_Projet:2N2222B, symbol Bibliotheque_Projet:2N2222B
Other:
- moved on the sheet: LS2
Changed lines of the file:
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@@
 	(symbol
 		(lib_id "Bibliotheque_Projet:CMT-8504-100-SMT-TR")
-		(at 240.03 113.03 0)
+		(at 232.41 82.55 0)
 		(unit 1)
 		(body_style 1)
@@
 		(fields_autoplaced yes)
 		(property "Reference" "LS2"
-			(at 256.54 105.41 0)
+			(at 248.92 74.93 0)
 			(show_name no)
 			(do_not_autoplace no)
@@
 		)
 		(property "Value" "CMT-8504-100-SMT-TR"
-			(at 256.54 107.95 0)
+			(at 248.92 77.47 0)
 			(show_name no)
 			(do_not_autoplace no)
@@
 		)
 		(property "Footprint" "Bibliotheque_Projet:Buzzer CMS"
-			(at 269.24 207.95 0)
+			(at 261.62 177.47 0)
 			(hide yes)
 			(show_name no)
@@
 		)
 		(property "Datasheet" "https://www.sameskydevices.com/product/resource/cmt-8504-100-smt-tr.pdf"
-			(at 269.24 307.95 0)
+			(at 261.62 277.47 0)
 			(hide yes)
 			(show_name no)
@@
 		)
 		(property "Description" "8.5 mm, 5 Vo-p, 100 dB, Surface Mount (SMT), Magnetic Audio Transducer Buzzer"
-			(at 240.03 113.03 0)
+			(at 232.41 82.55 0)
 			(hide yes)
 			(show_name no)
@@
 		)
 		(property "Height" "4.5"
-			(at 269.24 507.95 0)
+			(at 261.62 477.47 0)
 			(hide yes)
 			(show_name no)
@@
 		)
 		(property "Manufacturer_Name" "Same Sky"
-			(at 269.24 607.95 0)
+			(at 261.62 577.47 0)
 			(hide yes)
 			(show_name no)
@@
 		)
 		(property "Manufacturer_Part_Number" "CMT-8504-100-SMT-TR"
-			(at 269.24 707.95 0)
+			(at 261.62 677.47 0)
 			(hide yes)
 			(show_name no)
@@
 		)
 		(property "Mouser Part Number" "490-CMT-8504100SMTTR"
-			(at 269.24 807.95 0)
+			(at 261.62 777.47 0)
 			(hide yes)
 			(show_name no)
@@
 		)
 		(property "Mouser Price/Stock" "https://www.mouser.co.uk/ProductDetail/Same-Sky/CMT-8504-100-SMT-TR?qs=P1JMDcb91o7N%2FrNVZpuJrw%3D%3D"
-			(at 269.24 907.95 0)
+			(at 261.62 877.47 0)
 			(hide yes)
 			(show_name no)
@@
 		)
 		(property "Arrow Part Number" "CMT-8504-100-SMT-TR"
-			(at 269.24 1007.95 0)
+			(at 261.62 977.47 0)
 			(hide yes)
 			(show_name no)
@@
 		)
 		(property "Arrow Price/Stock" "https://www.arrow.com/en/products/cmt-8504-100-smt-tr/cui-devices.html?utm_currency=USD&region=nac"
-			(at 269.24 1107.95 0)
+			(at 261.62 1077.47 0)
 			(hide yes)
 			(show_name no)
@@
 				(path "/84605c1a-5009-408b-9a0f-13132cab7487"
 					(reference "LS2")
+					(unit 1)
+				)
+			)
+		)
+	)
+	(symbol
+		(lib_id "Bibliotheque_Projet:2N2222B")
+		(at 201.93 121.92 0)
+		(unit 1)
+		(body_style 1)
+		(exclude_from_sim no)
+		(in_bom yes)
+		(on_board yes)
+		(in_pos_files yes)
+		(dnp no)
+		(fields_autoplaced yes)
+		(property "Reference" "Q1"
+			(at 215.9 120.6499 0)
+			(show_name no)
+			(do_not_autoplace no)
+			(effects
+				(font
+					(size 1.27 1.27)
+				)
+				(justify left)
+			)
+		)
+		(property "Value" "2N2222B"
+			(at 215.9 123.1899 0)
+			(show_name no)
+			(do_not_autoplace no)
+			(effects
+				(font
+					(size 1.27 1.27)
+				)
+				(justify left)
+			)
+		)
+		(property "Footprint" "Bibliotheque_Projet:2N2222B"
+			(at 215.9 223.19 0)
+			(hide yes)
+			(show_name no)
+			(do_not_autoplace no)
+			(effects
+				(font
+					(size 1.27 1.27)
+				)
+				(justify left top)
+			)
+		)
+		(property "Datasheet" "https://diotec.com/request/datasheet/2n2222a.pdf"
+			(at 215.9 323.19 0)
+			(hide yes)
+			(show_name no)
+			(do_not_autoplace no)
+			(effects
+				(font
+					(size 1.27 1.27)
+				)
+				(justify left top)
+			)
+		)
+		(property "Description" "NPN General purpose transistor . IC 150 mA . f 	100 MHz"
+			(at 201.93 121.92 0)
+			(hide yes)
+			(show_name no)
+			(do_not_autoplace no)
+			(effects
+				(font
+					(size 1.27 1.27)
+				)
+			)
+		)
+		(property "Height" "7.5"
+			(at 215.9 523.19 0)
+			(hide yes)
+			(show_name no)
+			(do_not_autoplace no)
+			(effects
+				(font
+					(size 1.27 1.27)
+				)
+				(justify left top)
+			)
+		)
+		(property "Mouser Part Number" "637-2N2222A"
+			(at 215.9 623.19 0)
+			(hide yes)
+			(show_name no)
+			(do_not_autoplace no)
+			(effects
+				(font
+					(size 1.27 1.27)
+				)
+				(justify left top)
+			)
+		)
+		(property "Mouser Price/Stock" "https://www.mouser.co.uk/ProductDetail/Diotec-Semiconductor/2N2222A?qs=OlC7AqGiEDmNlRSTGL2dYg%3D%3D"
+			(at 215.9 723.19 0)
+			(hide yes)
+			(show_name no)
+			(do_not_autoplace no)
+			(effects
+				(font
+					(size 1.27 1.27)
+				)
+				(justify left top)
+			)
+		)
+		(property "Manufacturer_Name" "Diotec"
+			(at 215.9 823.19 0)
+			(hide yes)
+			(show_name no)
+			(do_not_autoplace no)
+			(effects
+				(font
+					(size 1.27 1.27)
+				)
+				(justify left top)
+			)
+		)
+		(property "Manufacturer_Part_Number" "2N2222A"
+			(at 215.9 923.19 0)
+			(hide yes)
+			(show_name no)
+			(do_not_autoplace no)
+			(effects
+				(font
+					(size 1.27 1.27)
+				)
+				(justify left top)
+			)
+		)
+		(pin "3"
+		)
+		(pin "1"
+		)
+		(pin "2"
+		)
+		(instances
+			(project "Ouvrier"
+				(path "/84605c1a-5009-408b-9a0f-13132cab7487"
+					(reference "Q1")
 					(unit 1)
 				)
@@
 	)
 	(symbol
-		(lib_id "power:+3V3")
-		(at 240.03 102.87 0)
-		(unit 1)
-		(body_style 1)
-		(exclude_from_sim no)
-		(in_bom yes)
-		(on_board yes)
-		(in_pos_files yes)
-		(dnp no)
-		(fields_autoplaced yes)
-		(property "Reference" "#PWR05"
-			(at 240.03 106.68 0)
-			(hide yes)
-			(show_name no)
-			(do_not_autoplace no)
-			(effects
-				(font
-					(size 1.27 1.27)
-				)
-			)
-		)
-		(property "Value" "+3V3"
-			(at 240.03 97.79 0)
-			(show_name no)
-			(do_not_autoplace no)
-			(effects
-				(font
-					(size 1.27 1.27)
-				)
-			)
-		)
-		(property "Footprint" ""
-			(at 240.03 102.87 0)
-			(hide yes)
-			(show_name no)
-			(do_not_autoplace no)
-			(effects
-				(font
-					(size 1.27 1.27)
-				)
-			)
-		)
-		(property "Datasheet" ""
-			(at 240.03 102.87 0)
-			(hide yes)
-			(show_name no)
-			(do_not_autoplace no)
-			(effects
-				(font
-					(size 1.27 1.27)
-				)
-			)
-		)
-		(property "Description" "Power symbol creates a global label with name \"+3V3\""
-			(at 240.03 102.87 0)
-			(hide yes)
-			(show_name no)
-			(do_not_autoplace no)
-			(effects
-				(font
-					(size 1.27 1.27)
-				)
-			)
-		)
-		(pin "1"
-		)
-		(instances
-			(project "Ouvrier"
-				(path "/84605c1a-5009-408b-9a0f-13132cab7487"
-					(reference "#PWR05")
-					(unit 1)
-				)
-			)
-		)
-	)
-	(symbol
 		(lib_id "Bibliotheque_Projet:XIAO-nRF52840-DIP")
 		(at 147.32 80.01 0)
@@
 					(unit 1)
 				)
-			)
-		)
-	)
-	(symbol
-		(lib_id "Transistor_BJT:2N2219")
-		(at 237.49 142.24 0)
-		(unit 1)
-		(body_style 1)
-		(exclude_from_sim no)
-		(in_bom yes)
-		(on_board yes)
-		(in_pos_files yes)
-		(dnp no)
-		(fields_autoplaced yes)
-		(property "Reference" "Q1"
-			(at 242.57 140.9699 0)
-			(show_name no)
-			(do_not_autoplace no)
-			(effects
-				(font
-					(size 1.27 1.27)
-				)
-				(justify left)
-			)
-		)
-		(property "Value" "2N2220"
-			(at 242.57 143.5099 0)
-			(show_name no)
-			(do_not_autoplace no)
-			(effects
-				(font
-					(size 1.27 1.27)
-				)
-				(justify left)
-			)
-		)
-		(property "Footprint" "Package_TO_SOT_THT:TO-39-3"
-			(at 242.57 144.145 0)
-			(hide yes)
-			(show_name no)
-			(do_not_autoplace no)
-			(effects
-				(font
-					(size 1.27 1.27)
-					(italic yes)
-				)
-				(justify left)
-			)
-		)
-		(property "Datasheet" "http://www.onsemi.com/pub_link/Collateral/2N2219-D.PDF"
-			(at 237.49 142.24 0)
-			(hide yes)
-			(show_name no)
-			(do_not_autoplace no)
-			(effects
-				(font
-					(size 1.27 1.27)
-				)
-				(justify left)
-			)
-		)
-		(property "Description" "800mA Ic, 50V Vce, NPN Transistor, TO-39"
-			(at 237.49 142.24 0)
-			(hide yes)
-			(show_name no)
-			(do_not_autoplace no)
-			(effects
-				(font
-					(size 1.27 1.27)
-				)
-			)
-		)
-		(property "Sim.Device" "NPN"
-			(at 237.49 142.24 0)
-			(hide yes)
-			(show_name no)
-			(do_not_autoplace no)
-			(effects
-				(font
-					(size 1.27 1.27)
-				)
-			)
-		)
-		(property "Sim.Pins" "1=E 2=B 3=C"
-			(at 237.49 142.24 0)
-			(hide yes)
-			(show_name no)
-			(do_not_autoplace no)
-			(effects
-				(font
-					(size 1.27 1.27)
-				)
-			)
-		)
-		(pin "3"
-		)
-		(pin "2"
-		)
-		(pin "1"
-		)
-		(instances
-			(project "Ouvrier"
-				(path "/84605c1a-5009-408b-9a0f-13132cab7487"
-					(reference "Q1")
-					(unit 1)
-				)

Commit message: MaJ batterie Ouvrier
Parts:
- added J1: Batterie, Bibliotheque_Projet:Batterie, symbol Bibliotheque_Projet:Batterie
Connections:
- net GNDREF: now also Q1.3 (C)
Other:
- moved on the sheet: D1, Q1
Changed lines of the file:
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@@
+	(wire
+		(pts
+			(xy 245.11 123.19) (xy 245.11 120.65)
+		)
+		(stroke
+			(width 0)
+			(type default)
+		)
+	)
 	(wire
 		(pts
@@
 		(pts
 			(xy 120.65 50.8) (xy 224.79 50.8)
+		)
+		(stroke
+			(width 0)
+			(type default)
+		)
+	)
+	(wire
+		(pts
+			(xy 245.11 120.65) (xy 251.46 120.65)
 		)
 		(stroke
@@
 	(symbol
 		(lib_id "Bibliotheque_Projet:2N2222B")
-		(at 201.93 121.92 0)
+		(at 234.95 130.81 0)
 		(unit 1)
 		(body_style 1)
@@
 		(fields_autoplaced yes)
 		(property "Reference" "Q1"
-			(at 215.9 120.6499 0)
+			(at 248.92 129.5399 0)
 			(show_name no)
 			(do_not_autoplace no)
@@
 		)
 		(property "Value" "2N2222B"
-			(at 215.9 123.1899 0)
+			(at 248.92 132.0799 0)
 			(show_name no)
 			(do_not_autoplace no)
@@
 		)
 		(property "Footprint" "Bibliotheque_Projet:2N2222B"
-			(at 215.9 223.19 0)
+			(at 248.92 232.08 0)
 			(hide yes)
 			(show_name no)
@@
 		)
 		(property "Datasheet" "https://diotec.com/request/datasheet/2n2222a.pdf"
-			(at 215.9 323.19 0)
+			(at 248.92 332.08 0)
 			(hide yes)
 			(show_name no)
@@
 		)
 		(property "Description" "NPN General purpose transistor . IC 150 mA . f 	100 MHz"
-			(at 201.93 121.92 0)
+			(at 234.95 130.81 0)
 			(hide yes)
 			(show_name no)
@@
 		)
 		(property "Height" "7.5"
-			(at 215.9 523.19 0)
+			(at 248.92 532.08 0)
 			(hide yes)
 			(show_name no)
@@
 		)
 		(property "Mouser Part Number" "637-2N2222A"
-			(at 215.9 623.19 0)
+			(at 248.92 632.08 0)
 			(hide yes)
 			(show_name no)
@@
 		)
 		(property "Mouser Price/Stock" "https://www.mouser.co.uk/ProductDetail/Diotec-Semiconductor/2N2222A?qs=OlC7AqGiEDmNlRSTGL2dYg%3D%3D"
-			(at 215.9 723.19 0)
+			(at 248.92 732.08 0)
 			(hide yes)
 			(show_name no)
@@
 		)
 		(property "Manufacturer_Name" "Diotec"
-			(at 215.9 823.19 0)
+			(at 248.92 832.08 0)
 			(hide yes)
 			(show_name no)
@@
 		)
 		(property "Manufacturer_Part_Number" "2N2222A"
-			(at 215.9 923.19 0)
+			(at 248.92 932.08 0)
 			(hide yes)
 			(show_name no)
@@
 				(path "/84605c1a-5009-408b-9a0f-13132cab7487"
 					(reference "Q1")
+					(unit 1)
+				)
+			)
+		)
+	)
+	(symbol
+		(lib_id "Bibliotheque_Projet:Batterie")
+		(at 246.38 105.41 0)
+		(unit 1)
+		(body_style 1)
+		(exclude_from_sim no)
+		(in_bom yes)
+		(on_board yes)
+		(in_pos_files yes)
+		(dnp no)
+		(fields_autoplaced yes)
+		(property "Reference" "J1"
+			(at 247.015 100.33 0)
+			(show_name no)
+			(do_not_autoplace no)
+			(effects
+				(font
+					(size 1.27 1.27)
+				)
+			)
+		)
+		(property "Value" "Batterie"
+			(at 247.015 102.87 0)
+			(show_name no)
+			(do_not_autoplace no)
+			(effects
+				(font
+					(size 1.27 1.27)
+				)
+			)
+		)
+		(property "Footprint" "Bibliotheque_Projet:Batterie"
+			(at 249.682 103.378 0)
+			(hide yes)
+			(show_name no)
+			(do_not_autoplace no)
+			(effects
+				(font
+					(size 1.27 1.27)
+				)
+			)
+		)
+		(property "Datasheet" ""
+			(at 246.38 105.41 0)
+			(hide yes)
+			(show_name no)
+			(do_not_autoplace no)
+			(effects
+				(font
+					(size 1.27 1.27)
+				)
+			)
+		)
+		(property "Description" "Pads batterie"
+			(at 249.682 100.838 0)
+			(hide yes)
+			(show_name no)
+			(do_not_autoplace no)
+			(effects
+				(font
+					(size 1.27 1.27)
+				)
+			)
+		)
+		(pin "Bat-"
+		)
+		(pin "Bat+"
+		)
+		(instances
+			(project "Ouvrier"
+				(path "/84605c1a-5009-408b-9a0f-13132cab7487"
+					(reference "J1")
 					(unit 1)
 				)
@@
 	(symbol
 		(lib_id "power:GNDREF")
-		(at 240.03 151.13 0)
+		(at 251.46 120.65 0)
 		(unit 1)
 		(body_style 1)
@@
 		(fields_autoplaced yes)
 		(property "Reference" "#PWR02"
-			(at 240.03 157.48 0)
+			(at 251.46 127 0)
 			(hide yes)
 			(show_name no)
@@
 		)
 		(property "Value" "GNDREF"
-			(at 240.03 156.21 0)
+			(at 251.46 125.73 0)
 			(show_name no)
 			(do_not_autoplace no)
@@
 		)
 		(property "Footprint" ""
-			(at 240.03 151.13 0)
+			(at 251.46 120.65 0)
 			(hide yes)
 			(show_name no)
@@
 		)
 		(property "Datasheet" ""
-			(at 240.03 151.13 0)
+			(at 251.46 120.65 0)
 			(hide yes)
 			(show_name no)
@@
 		)
 		(property "Description" "Power symbol creates a global label with name \"GNDREF\" , reference supply ground"
-			(at 240.03 151.13 0)
+			(at 251.46 120.65 0)
 			(hide yes)
 			(show_name no)
@@
 	(symbol
 		(lib_id "Diode:1N914")
-		(at 232.41 123.19 270)
+		(at 223.52 83.82 270)
 		(unit 1)
 		(body_style 1)
@@
 		(fields_autoplaced yes)
 		(property "Reference" "D1"
-			(at 234.95 121.9199 90)
+			(at 226.06 82.5499 90)
 			(show_name no)
 			(do_not_autoplace no)
@@
 		)
 		(property "Value" "1N914"
-			(at 234.95 124.4599 90)
+			(at 226.06 85.0899 90)
 			(show_name no)
 			(do_not_autoplace no)
@@
 		)
 		(property "Footprint" "Diode_THT:D_DO-35_SOD27_P7.62mm_Horizontal"
-			(at 227.965 123.19 0)
+			(at 219.075 83.82 0)
 			(hide yes)
 			(show_name no)
@@
 		)
 		(property "Datasheet" "http://www.vishay.com/docs/85622/1n914.pdf"
-			(at 232.41 123.19 0)
+			(at 223.52 83.82 0)
 			(hide yes)
 			(show_name no)
@@
 		)
 		(property "Description" "100V 0.3A Small Signal Fast Switching Diode, DO-35"
-			(at 232.41 123.19 0)
+			(at 223.52 83.82 0)
 			(hide yes)
 			(show_name no)
@@
 		)
 		(property "Sim.Device" "D"
-			(at 232.41 123.19 0)
+			(at 223.52 83.82 0)
 			(hide yes)
 			(show_name no)
@@
 		)
 		(property "Sim.Pins" "1=K 2=A"
-			(at 232.41 123.19 0)
-			(hide yes)
-			(show_name no)
+			(at 223.52 83.82 0)
+			(hide yes)
+			(show_name no)

Commit message: ouvrier
Connections:
- net +3V3: now also D1.1 (K), J1.Bat+ (Pin_2), LS2.1 (+)
- net GNDREF: now also J1.Bat- (Pin_1), Q1.1 (E); no longer Q1.3 (C)
- net at R1.1: now also U1.3 (P0.28_A2_D2)
- net at R1.2: now also Q1.2 (B)
- net at LS2.2 (-): now also D1.2 (A), Q1.3 (C)
Other:
- moved on the sheet: D1, LS2, Q1, R1

Commit message: Ouvrier_v3_fini
Parts:
- added C1: 100nF, Capacitor_SMD:C_0402_1005Metric_Pad0.74x0.62mm_HandSolder, symbol Device:C
- R1: value 180 -> 470
Connections:
- net +3V3: now also C1.1
- net GNDREF: now also C1.2

Commit message: Ouvrier_v5_valeurR1
Parts:
- R1: value 470 -> 680
Changed lines of the file:
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@@
 			)
 		)
-		(property "Value" "470"
+		(property "Value" "680"
 			(at 212.09 133.35 90)
 			(show_name no)
