File: PCB/Ouvrier/Ouvrier.kicad_pcb (KiCad board)
At the start: 2 copper layers, 7 parts, among them Q1 2N2220, U1 XIAO-ESP32-S3-Plus-DIP, U2 BMP581, U3 UWB

Commit message: MaJ batterie KiCad Ouvrier
Parts:
- Q1: value 2N2220 -> 2N2222B; footprint Package_TO_SOT_THT:TO-39-3 -> Bibliotheque_Projet:2N2222B
- moved Q1 3.15 mm to (149.5, 96.5)
- moved U2 1.78 mm to (145.5, 103.5)

Commit message: MaJ batterie Ouvrier
Parts:
- added J1: Batterie, Bibliotheque_Projet:Batterie, F.Cu at (152.0, 101.0)
Changed lines of the file:
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@@
 		)
+	)
+	(footprint "Bibliotheque_Projet:Batterie"
+		(layer "F.Cu")
+		(at 152 101)
+		(property "Reference" "J1"
+			(at 0 -0.5 0)
+			(unlocked yes)
+			(layer "F.SilkS")
+			(effects
+				(font
+					(size 1 1)
+					(thickness 0.1)
+				)
+			)
+		)
+		(property "Value" "Batterie"
+			(at 0 1 0)
+			(unlocked yes)
+			(layer "F.Fab")
+			(effects
+				(font
+					(size 1 1)
+					(thickness 0.15)
+				)
+			)
+		)
+		(property "Datasheet" ""
+			(at 0 0 0)
+			(unlocked yes)
+			(layer "F.Fab")
+			(hide yes)
+			(effects
+				(font
+					(size 1 1)
+					(thickness 0.15)
+				)
+			)
+		)
+		(property "Description" "Pads batterie"
+			(at 0 0 0)
+			(unlocked yes)
+			(layer "F.Fab")
+			(hide yes)
+			(effects
+				(font
+					(size 1 1)
+					(thickness 0.15)
+				)
+			)
+		)
+		(property ki_fp_filters "Connector*:*_1x??_*")
+		(sheetname "/")
+		(sheetfile "Ouvrier.kicad_sch")
+		(units
+			(unit
+				(name "A")
+				(pins "Bat-" "Bat+")
+			)
+		)
+		(duplicate_pad_numbers_are_jumpers no)
+		(fp_rect
+			(start -4 4)
+			(end 4 9.5)
+			(stroke
+				(width 0.1)
+				(type default)
+			)
+			(fill no)
+			(layer "F.SilkS")
+		)
+		(fp_text user "Bat-"
+			(at 0 6 0)
+			(unlocked yes)
+			(layer "F.SilkS")
+			(effects
+				(font
+					(size 1 1)
+					(thickness 0.1)
+				)
+				(justify left bottom)
+			)
+		)
+		(fp_text user "Bat+"
+			(at 0 8.5 0)
+			(unlocked yes)
+			(layer "F.SilkS")
+			(effects
+				(font
+					(size 1 1)
+					(thickness 0.1)
+				)
+				(justify left bottom)
+			)
+		)
+		(fp_text user "${REFERENCE}"
+			(at 0 2.5 0)
+			(unlocked yes)
+			(layer "F.Fab")
+			(effects
+				(font
+					(size 1 1)
+					(thickness 0.15)
+				)
+			)
+		)
+		(pad "Bat+" thru_hole roundrect
+			(at -1 8)
+			(size 3.27 1.27)
+			(drill 0.8
+				(offset -1 0)
+			)
+			(layers "*.Cu" "*.Mask")
+			(remove_unused_layers no)
+			(roundrect_rratio 0.15)
+			(net "unconnected-(J1-Pin_2-PadBat+)")
+			(pinfunction "Pin_2_Bat+")
+			(pintype "passive")
+		)
+		(pad "Bat-" thru_hole roundrect
+			(at -1 5.5)
+			(size 3.27 1.27)
+			(drill 0.8
+				(offset -1 0)
+			)
+			(layers "*.Cu" "*.Mask")
+			(remove_unused_layers no)
+			(roundrect_rratio 0.15)
+			(net "unconnected-(J1-Pin_1-PadBat-)")
+			(pinfunction "Pin_1_Bat-")
+			(pintype "passive")
+		)
+		(embedded_fonts no)
 	)
 	(footprint "Bibliotheque_Projet:XIAO nRF52840 sense plus"

Commit message: ouvrier
Connections:
- D1 pad 1: unconnected-(D1-K-Pad1) -> +3V3
- D1 pad 2: unconnected-(D1-A-Pad2) -> Net-(D1-A)
- J1 pad Bat+: unconnected-(J1-Pin_2-PadBat+) -> +3V3
- J1 pad Bat-: unconnected-(J1-Pin_1-PadBat-) -> GNDREF
- LS2 pad 1: unconnected-(LS2-+-Pad1) -> +3V3
- LS2 pad 2: unconnected-(LS2---Pad2) -> Net-(D1-A)
- Q1 pad 1: unconnected-(Q1-E-Pad1) -> GNDREF
- Q1 pad 2: unconnected-(Q1-B-Pad2) -> Net-(Q1-B)
- Q1 pad 3: unconnected-(Q1-C-Pad3) -> Net-(D1-A)
- R1 pad 1: unconnected-(R1-Pad1) -> Net-(U1-P0.28_A2_D2)
- R1 pad 2: unconnected-(R1-Pad2) -> Net-(Q1-B)
- U1 pad 3: unconnected-(U1-P0.28_A2_D2-Pad3) -> Net-(U1-P0.28_A2_D2)
Changed lines of the file:
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@@
 			(size 2.5 2.5)
 			(layers "F.Cu" "F.Mask" "F.Paste")
-			(net "unconnected-(LS2-+-Pad1)")
+			(net "+3V3")
 			(pinfunction "+_1")
 			(pintype "passive")
@@
 			(size 2.5 2.5)
 			(layers "F.Cu" "F.Mask" "F.Paste")
-			(net "unconnected-(LS2---Pad2)")
+			(net "Net-(D1-A)")
 			(pinfunction "-_2")
 			(pintype "passive")
@@
 			(remove_unused_layers no)
 			(roundrect_rratio 0.15)
-			(net "unconnected-(J1-Pin_2-PadBat+)")
+			(net "+3V3")
 			(pinfunction "Pin_2_Bat+")
 			(pintype "passive")
@@
 			(remove_unused_layers no)
 			(roundrect_rratio 0.15)
-			(net "unconnected-(J1-Pin_1-PadBat-)")
+			(net "GNDREF")
 			(pinfunction "Pin_1_Bat-")
 			(pintype "passive")
@@
 			(layers "F.Cu" "F.Mask")
 			(roundrect_rratio 0.1)
-			(net "unconnected-(U1-P0.28_A2_D2-Pad3)")
+			(net "Net-(U1-P0.28_A2_D2)")
 			(pinfunction "P0.28_A2_D2_3")
 			(pintype "passive")
@@
 			(layers "*.Cu" "*.Mask")
 			(remove_unused_layers no)
-			(net "unconnected-(U1-P0.28_A2_D2-Pad3)")
+			(net "Net-(U1-P0.28_A2_D2)")
 			(pinfunction "P0.28_A2_D2_3")
 			(pintype "passive")
@@
 			(remove_unused_layers no)
 			(roundrect_rratio 0.15625)
-			(net "unconnected-(D1-K-Pad1)")
+			(net "+3V3")
 			(pinfunction "K_1")
 			(pintype "passive")
@@
 			(layers "*.Cu" "*.Mask")
 			(remove_unused_layers no)
-			(net "unconnected-(D1-A-Pad2)")
+			(net "Net-(D1-A)")
 			(pinfunction "A_2")
 			(pintype "passive")
@@
 			(layers "*.Cu" "*.Mask")
 			(remove_unused_layers no)
-			(net "unconnected-(Q1-E-Pad1)")
+			(net "GNDREF")
 			(pinfunction "E_1")
 			(pintype "passive")
@@
 			(layers "*.Cu" "*.Mask")
 			(remove_unused_layers no)
-			(net "unconnected-(Q1-B-Pad2)")
+			(net "Net-(Q1-B)")
 			(pinfunction "B_2")
 			(pintype "passive")
@@
 			(layers "*.Cu" "*.Mask")
 			(remove_unused_layers no)
-			(net "unconnected-(Q1-C-Pad3)")
+			(net "Net-(D1-A)")
 			(pinfunction "C_3")
 			(pintype "passive")
@@
 			(layers "*.Cu" "*.Mask")
 			(remove_unused_layers no)
-			(net "unconnected-(R1-Pad1)")
+			(net "Net-(U1-P0.28_A2_D2)")
 			(pintype "passive")
 		)
@@
 			(layers "*.Cu" "*.Mask")
 			(remove_unused_layers no)
-			(net "unconnected-(R1-Pad2)")
-			(pintype "passive")
-		)
+			(net "Net-(Q1-B)")
+			(pintype "passive")
+		)

Commit message: Ouvrier_v2
Parts:
- added REF**: MountingHole_3.2mm_M3, MountingHole:MountingHole_3.2mm_M3, F.Cu at (99.0, 106.0)
- added REF**: MountingHole_3.2mm_M3, MountingHole:MountingHole_3.2mm_M3, F.Cu at (140.0, 60.0)
- added REF**: MountingHole_3.2mm_M3, MountingHole:MountingHole_3.2mm_M3, F.Cu at (99.0, 60.0)
- added REF**: MountingHole_3.2mm_M3, MountingHole:MountingHole_3.2mm_M3, F.Cu at (140.0, 106.0)
- moved J1 53.3 mm to (99.5, 91.6)
- moved Q1 36.1 mm to (113.5, 99.8), turned to 90 degrees
- moved U3 35.4 mm to (118.2, 64.8), turned to 180 degrees
- moved R1 17.5 mm to (120.0, 88.2), turned to -90 degrees
- moved U2 15.0 mm to (138.5, 90.2), turned to 90 degrees
- moved D1 12.9 mm to (123.2, 88.7), turned to -90 degrees
- moved U1 11.4 mm to (131.5, 76.6), turned to 90 degrees
- moved LS2 7.63 mm to (130.5, 93.8)
Routing:
- net +3V3: track 0.00 -> 176.0 mm
- net GNDREF: track 0.00 -> 86.8 mm
- net Net-(U1-P1.14_D9_MISO): track 0.00 -> 45.6 mm
- net Net-(U1-P1.12_D7_RX): track 0.00 -> 43.4 mm, vias 0 -> 1
- net Net-(U1-P0.29_A3_D3): track 0.00 -> 26.9 mm
- net Net-(U1-P1.11_D6_TX): track 0.00 -> 26.3 mm
- net Net-(U1-P1.15_D10_MOSI): track 0.00 -> 20.0 mm
- net Net-(U1-P0.28_A2_D2): track 0.00 -> 17.0 mm
- net Net-(U1-P1.13_D8_SCK): track 0.00 -> 16.5 mm
- net Net-(D1-A): track 0.00 -> 14.3 mm
- net Net-(U1-P0.02_A0_D0): track 0.00 -> 13.7 mm
- net Net-(Q1-B): track 0.00 -> 7.87 mm
- added copper zone on B.Cu, net GNDREF
Other:
- board outline added: 52 x 54.5 mm
- board text added: "VIGIZONE 2026 ESIEE PARIS"

Commit message: Ouvrier_v3_fini
Parts:
- added C1: 100nF, Capacitor_SMD:C_0402_1005Metric_Pad0.74x0.62mm_HandSolder, F.Cu at (136.9, 93.0)
- R1: value 180 -> 470
Routing:
- net Net-(U1-P1.12_D7_RX): track 43.4 -> 46.8 mm
- net +3V3: track 176.0 -> 174.6 mm
Other:
- board text added: "BLONDEL.C ESIEE PARIS 2026"
- board text removed: "VIGIZONE 2026 ESIEE PARIS"

Commit message: Ouvrier_v4_test_DRC
Parts:
- moved C1 0.55 mm to (137.4, 93.0)
Routing:
- net +3V3: track 174.6 -> 178.1 mm
- net GNDREF: track 86.8 -> 88.8 mm, vias 0 -> 1
- net Net-(U1-P1.13_D8_SCK): track 16.5 -> 18.2 mm

Commit message: batterie et Induction
Parts:
- added J2: VBAT Xiao, Bibliotheque_Projet:Raccord VBat XIAO, F.Cu at (137.4, 72.5)
- added J3: DC 5V input, Bibliotheque_Projet:chargeur sans fil, F.Cu at (141.0, 63.5)
- R1: value 470 -> 680
- moved J1 37.1 mm to (122.2, 62.2), turned to -90 degrees
Connections:
- J1 pad Bat+: +3V3 -> Net-(J1-Pin_2)
- J1 pad Bat-: GNDREF -> Net-(J1-Pin_1)
- U1 pad 13: unconnected-(U1-GND-Pad13) -> Net-(U1-GND)
- U1 pad 14: unconnected-(U1-VBUS-Pad14) -> Net-(U1-VBUS)
Routing:
- net Net-(J1-Pin_1): track 0.00 -> 28.7 mm
- net Net-(J1-Pin_2): track 0.00 -> 28.7 mm
- net Net-(U1-GND): track 0.00 -> 2.41 mm, vias 0 -> 1

Commit message: ouvrier_v6
Connections:
- net Net-(U1-VBUS) renamed +5V
- J3 pad GND: Net-(U1-GND) -> GNDREF
- U1 pad 13: Net-(U1-GND) -> GNDREF
Routing:
- net +3V3: track 178.1 -> 92.1 mm
- net GNDREF: track 88.8 -> 58.7 mm
- net Net-(U1-GND): track 2.41 -> 0.00 mm, vias 1 -> 0
- net Net-(U1-P1.12_D7_RX): track 46.5 -> 45.3 mm
