File: PCB/Ouvrier/Ouvrier.kicad_pcb (KiCad board)
At the start: 2 copper layers, 52 x 54.5 mm, 15 parts, among them J1 Batterie, J2 VBAT Xiao, J3 DC 5V input, Q1 2N2222B, U1 XIAO-ESP32-S3-Plus-DIP, U2 BMP581, U3 UWB

Commit message: led ouvrier kicad
Parts:
- added D2: LED, Bibliotheque_Projet:LED_D3.0mm_Clear, F.Cu at (141.0, 96.7)
- added R3: 330R, Resistor_THT:R_Axial_DIN0207_L6.3mm_D2.5mm_P10.16mm_Horizontal, F.Cu at (129.9, 74.4)
Connections:
- U1 pad 5: unconnected-(U1-P0.04_A4_D4_SDA-Pad5) -> Net-(U1-P0.04_A4_D4_SDA)

Commit message: Ouvrier_v7
Routing:
- net Net-(J1-Pin_2): track 28.7 -> 25.5 mm
- net Net-(J1-Pin_1): track 28.7 -> 25.6 mm
Changed lines of the file:
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@@
 	)
 	(segment
-		(start 130.9 67.4)
-		(end 130.9 72.5)
+		(start 114.5 64)
+		(end 123.5 64)
 		(width 0.8)
 		(layer "F.Cu")
@@
 	)
 	(segment
-		(start 114.5 64)
-		(end 118.5 64)
+		(start 126 66.5)
+		(end 130 66.5)
 		(width 0.8)
 		(layer "F.Cu")
@@
 	)
 	(segment
-		(start 123.5 62)
-		(end 123.5 64)
+		(start 130 66.5)
+		(end 130.9 67.4)
+		(width 0.8)
+		(layer "F.Cu")
+		(net "Net-(J1-Pin_2)")
+	)
+	(segment
+		(start 130.9 67.4)
+		(end 130.9 72.5)
 		(width 0.8)
 		(layer "F.Cu")
@@
 	)
 	(segment
-		(start 130 66.5)
-		(end 130.9 67.4)
-		(width 0.8)
-		(layer "F.Cu")
-		(net "Net-(J1-Pin_2)")
-	)
-	(segment
-		(start 121 61.5)
-		(end 123 61.5)
-		(width 0.8)
-		(layer "F.Cu")
-		(net "Net-(J1-Pin_2)")
-	)
-	(segment
-		(start 123 61.5)
-		(end 123.5 62)
-		(width 0.8)
-		(layer "F.Cu")
-		(net "Net-(J1-Pin_2)")
-	)
-	(segment
-		(start 126 66.5)
-		(end 130 66.5)
-		(width 0.8)
-		(layer "F.Cu")
-		(net "Net-(J1-Pin_2)")
-	)
-	(segment
 		(start 112.75 62.25)
 		(end 114.5 64)
-		(width 0.8)
-		(layer "F.Cu")
-		(net "Net-(J1-Pin_2)")
-	)
-	(segment
-		(start 118.5 64)
-		(end 121 61.5)
 		(width 0.8)
 		(layer "F.Cu")
@@
 	)
 	(segment
-		(start 125 61.25)
-		(end 125 63.125)
-		(width 0.8)
-		(layer "F.Cu")
-		(net "Net-(J1-Pin_1)")
-	)
-	(segment
-		(start 123.75 60)
-		(end 125 61.25)
-		(width 0.8)
-		(layer "F.Cu")
-		(net "Net-(J1-Pin_1)")
-	)
-	(segment
-		(start 115.4 62.5)
-		(end 118 62.5)
-		(width 0.8)
-		(layer "F.Cu")
-		(net "Net-(J1-Pin_1)")
-	)
-	(segment
-		(start 120.5 60)
-		(end 123.75 60)
-		(width 0.8)
-		(layer "F.Cu")
-		(net "Net-(J1-Pin_1)")
-	)
-	(segment
-		(start 125 63.125)
-		(end 126.875 65)
-		(width 0.8)
-		(layer "F.Cu")
-		(net "Net-(J1-Pin_1)")
-	)
-	(segment
 		(start 131.5 65)
 		(end 132.9 66.4)
@@
 	)
 	(segment
-		(start 126.875 65)
-		(end 131.5 65)
+		(start 115.15 62.25)
+		(end 115.4 62.5)
+		(width 0.8)
+		(layer "F.Cu")
+		(net "Net-(J1-Pin_1)")
+	)
+	(segment
+		(start 115.4 62.5)
+		(end 124.375 62.5)
 		(width 0.8)
 		(layer "F.Cu")
@@
 	)
 	(segment
-		(start 118 62.5)
-		(end 120.5 60)
+		(start 124.375 62.5)
+		(end 126.875 65)
 		(width 0.8)
 		(layer "F.Cu")
@@
 	)
 	(segment
-		(start 115.15 62.25)
-		(end 115.4 62.5)
+		(start 126.875 65)
+		(end 131.5 65)
 		(width 0.8)
 		(layer "F.Cu")

Commit message: Ouvrier_v7
Parts:
- moved R3 40.7 mm to (96.2, 97.2), turned to 0 degrees
- moved J3 37.8 mm to (103.5, 58.8), turned to 90 degrees
- moved J1 18.1 mm to (140.3, 61.5)
- moved D2 2.54 mm to (141.0, 99.3), turned to 90 degrees
- moved D1 0.75 mm to (123.2, 89.4)
- moved R1 0.75 mm to (120.0, 88.9)
Routing:
- net Net-(D2-K): track 0.00 -> 44.3 mm
- net Net-(U1-P0.04_A4_D4_SDA): track 0.00 -> 42.9 mm
- net +5V: track 0.00 -> 29.6 mm
- net Net-(J1-Pin_1): track 25.6 -> 11.1 mm
- net Net-(J1-Pin_2): track 25.5 -> 11.3 mm
- net GNDREF: track 58.7 -> 71.5 mm
- net Net-(U1-P0.28_A2_D2): track 17.0 -> 23.1 mm
- net Net-(U1-P1.12_D7_RX): track 45.3 -> 42.3 mm
- net +3V3: track 92.1 -> 92.9 mm
- net Net-(D1-A): track 14.3 -> 15.0 mm
