File: PCB/Ancre/Ancre.kicad_pcb (KiCad board)
At the start: 2 copper layers, 72.2 x 60.7 mm, 17 parts, among them IC1 TCAN1051VDRQ1, U1 OKI-78SR-5_1.5-W36-C, U2 DB301V-5.0-2P, U3 DB301V-5.0-2P, U6 DB301V-5.0-2P, U7 DB301V-5.0-2P

Commit message: ancre fini ?
Parts:
- added C5: 100nF, Capacitor_THT:C_Axial_L3.8mm_D2.6mm_P7.50mm_Horizontal, F.Cu at (253.0, 80.0)
- moved IC1 2.00 mm to (249.0, 84.5)
- moved U1 0.50 mm to (258.0, 87.0)
Routing:
- net Net-(IC1-TXD): track 35.1 -> 38.0 mm
- net Net-(IC1-CANL): track 39.0 -> 36.5 mm
- net Net-(IC1-NC): track 46.9 -> 48.9 mm
- net Net-(IC1-RXD): track 33.6 -> 35.5 mm
- net Net-(IC1-S): track 20.7 -> 18.8 mm
- net GNDREF: track 13.3 -> 11.7 mm
- net Net-(IC1-CANH): track 23.8 -> 22.2 mm
- net +5V: track 47.5 -> 46.7 mm
- net +12V: track 26.7 -> 26.0 mm

Commit message: Ancre_v12_fini
Parts:
- C1: value C -> 10uF
Routing:
- net Net-(IC1-NC): track 48.9 -> 51.1 mm
- net Net-(IC1-RXD): track 35.5 -> 36.9 mm
- net Net-(IC1-TXD): track 38.0 -> 38.5 mm
Changed lines of the file:
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@@
 			)
 		)
-		(property "Value" "C"
+		(property "Value" "10uF"
 			(at -8.21 2.19 90)
 			(layer "F.Fab")
@@
 			(font
 				(size 1.5 1.5)
-				(thickness 0.3)
+				(thickness 0.375)
 				(bold yes)
 			)
@@
 	)
 	(segment
-		(start 249.546961 77.9832)
-		(end 250.030161 77.5)
+		(start 240.1 77.51)
+		(end 240.11 77.5)
+		(width 0.8)
+		(layer "F.Cu")
+		(net "+5V")
+	)
+	(segment
+		(start 254.88 77.5)
+		(end 258.02 80.64)
 		(width 0.8)
 		(layer "F.Cu")
@@
 	)
 	(segment
-		(start 241.985882 77.7832)
-		(end 248.433039 77.7832)
+		(start 258.02 80.64)
+		(end 258.02 81.97)
 		(width 0.8)
 		(layer "F.Cu")
@@
 	)
 	(segment
-		(start 250.030161 77.5)
+		(start 240.11 77.5)
 		(end 254.88 77.5)
 		(width 0.8)
@@
 	)
 	(segment
-		(start 254.88 77.5)
-		(end 258.02 80.64)
-		(width 0.8)
-		(layer "F.Cu")
-		(net "+5V")
-	)
-	(segment
-		(start 241.702682 77.5)
-		(end 241.985882 77.7832)
-		(width 0.8)
-		(layer "F.Cu")
-		(net "+5V")
-	)
-	(segment
-		(start 248.633039 77.9832)
-		(end 249.546961 77.9832)
-		(width 0.8)
-		(layer "F.Cu")
-		(net "+5V")
-	)
-	(segment
-		(start 240.1 77.51)
-		(end 240.11 77.5)
-		(width 0.8)
-		(layer "F.Cu")
-		(net "+5V")
-	)
-	(segment
 		(start 255.32 84.2)
 		(end 254.985 83.865)
@@
 	)
 	(segment
-		(start 240.11 77.5)
-		(end 241.702682 77.5)
+		(start 254.985 83.865)
+		(end 251.711 83.865)
 		(width 0.8)
 		(layer "F.Cu")
@@
 	)
 	(segment
-		(start 258.02 80.64)
-		(end 258.02 81.97)
-		(width 0.8)
-		(layer "F.Cu")
-		(net "+5V")
+		(start 240.86 83.03)
+		(end 239.32 84.57)
+		(width 0.6)
+		(layer "B.Cu")
+		(net "Net-(U5-Resistance)")
 	)
 	(segment
-		(start 248.433039 77.7832)
-		(end 248.633039 77.9832)
-		(width 0.8)
-		(layer "F.Cu")
-		(net "+5V")
+		(start 240.86 79.72)
+		(end 240.86 83.03)
+		(width 0.6)
+		(layer "B.Cu")
+		(net "Net-(U5-Resistance)")
 	)
 	(segment
-		(start 254.985 83.865)
-		(end 251.711 83.865)
-		(width 0.8)
-		(layer "F.Cu")
-		(net "+5V")
+		(start 239.32 84.57)
+		(end 233.89 84.57)
+		(width 0.6)
+		(layer "B.Cu")
+		(net "Net-(U5-Resistance)")
+	)
+	(segment
+		(start 233.89 84.57)
+		(end 228.46 90)
+		(width 0.6)
+		(layer "B.Cu")
+		(net "Net-(U5-Resistance)")
 	)
 	(segment
@@
 	)
 	(segment
-		(start 242.36 76.88)
-		(end 249.09 76.88)
+		(start 240.67 75.19)
+		(end 240.67 73.4)
 		(width 0.6)
 		(layer "F.Cu")
@@
 	)
 	(segment
-		(start 228.8 73.12)
+		(start 240.67 73.4)
 		(end 240.39 73.12)
 		(width 0.6)
@@
 	)
 	(segment
-		(start 227.88 74.04)
-		(end 228.8 73.12)
+		(start 249 85.5)
+		(end 249.905 86.405)
 		(width 0.6)
 		(layer "F.Cu")
@@
 	)
 	(segment
-		(start 249 85.5)
-		(end 249.905 86.405)
+		(start 227.88 74.04)
+		(end 227.88 76.1)
 		(width 0.6)
 		(layer "F.Cu")
@@
 	)
 	(segment
-		(start 240.67 75.19)
-		(end 242.36 76.88)
+		(start 228.8 73.12)
+		(end 227.88 74.04)
 		(width 0.6)
 		(layer "F.Cu")
@@
 	)
 	(segment
-		(start 240.67 73.4)
-		(end 240.67 75.19)
+		(start 240.39 73.12)
+		(end 228.8 73.12)
 		(width 0.6)
 		(layer "F.Cu")
@@
 	)
 	(segment
-		(start 240.39 73.12)
-		(end 240.67 73.4)
+		(start 241.48 76)
+		(end 240.67 75.19)
 		(width 0.6)
 		(layer "F.Cu")
@@
 	)
 	(segment
-		(start 227.88 76.1)
-		(end 227.88 74.04)
+		(start 249.09 76)
+		(end 241.48 76)
 		(width 0.6)
 		(layer "F.Cu")
@@
 	)
 	(via
-		(at 249.09 76.88)
+		(at 249.09 76)
 		(size 1)
 		(drill 0.8)
@@
 	)
 	(segment
-		(start 249.09 83.91)
-		(end 249 84)
+		(start 249.09 76)
+		(end 249.09 83.91)
 		(width 0.6)
 		(layer "B.Cu")
@@
 	)
 	(segment
-		(start 249.09 76.88)
-		(end 249.09 83.91)
+		(start 249.09 83.91)
+		(end 249 84)
 		(width 0.6)
 		(layer "B.Cu")
@@
 	)
 	(segment
-		(start 255.55 81.56)
-		(end 254.515 82.595)
+		(start 255.55 76.955)
+		(end 251.595 73)
 		(width 0.6)
 		(layer "B.Cu")
@@
 	)
 	(segment
-		(start 231.96 74.56)
-		(end 230.42 76.1)
+		(start 253.5 82.595)
+		(end 254.515 82.595)
 		(width 0.6)
 		(layer "B.Cu")
@@
 	)
 	(segment
-		(start 253 74.63)
-		(end 255.55 77.18)
+		(start 251.595 73)
+		(end 233.52 73)
 		(width 0.6)
 		(layer "B.Cu")
@@
 	)
 	(segment
-		(start 253 74.63)
-		(end 253 74.56)
-		(width 0.2)
+		(start 233.52 73)
+		(end 230.42 76.1)
+		(width 0.6)
 		(layer "B.Cu")
 		(net "Net-(IC1-RXD)")
 	)
 	(segment
-		(start 253 74.56)
-		(end 231.96 74.56)
+		(start 254.515 82.595)
+		(end 255.55 81.56)
 		(width 0.6)
 		(layer "B.Cu")
@@
 	)
 	(segment
-		(start 255.55 77.18)
-		(end 255.55 81.56)
+		(start 255.55 81.56)
+		(end 255.55 76.955)
 		(width 0.6)
 		(layer "B.Cu")
@@
 	)
 	(segment
-		(start 254.515 82.595)
-		(end 253.5 82.595)
+		(start 245.5 80)
+		(end 245.5 80.5)
+		(width 0.2)
+		(layer "F.Cu")
+		(net "Net-(IC1-NC)")
+	)
+	(segment
+		(start 244.595 82.595)
+		(end 246.289 82.595)
 		(width 0.6)
-		(layer "B.Cu")
-		(net "Net-(IC1-RXD)")
+		(layer "F.Cu")
+		(net "Net-(IC1-NC)")
 	)
 	(segment
-		(start 243.24 75.62)
-		(end 243.24 53.37)
+		(start 244.5 80)
+		(end 244 80)
 		(width 0.6)
 		(layer "F.Cu")
@@
 	(segment
 		(start 245.5 80)
-		(end 245.5 80.5)
-		(width 0.2)
+		(end 244.5 80)
+		(width 0.6)
 		(layer "F.Cu")
 		(net "Net-(IC1-NC)")
 	)
 	(segment
-		(start 245.5 80)
-		(end 244 80)
+		(start 243.24 53.37)
+		(end 246.57 50.04)
 		(width 0.6)
 		(layer "F.Cu")
@@
 	)
 	(segment
-		(start 246.57 50.04)
-		(end 255.67 50.04)
+		(start 244 80)
+		(end 244 80.75)
 		(width 0.6)
 		(layer "F.Cu")
@@
 	)
 	(segment
-		(start 245.5 80.5)
-		(end 246.289 81.289)
+		(start 244 82)
+		(end 244.595 82.595)
 		(width 0.6)
 		(layer "F.Cu")
@@
 	)
 	(segment
-		(start 243.24 53.37)
-		(end 246.57 50.04)
+		(start 243.24 74.5)
+		(end 243.24 53.37)
 		(width 0.6)
 		(layer "F.Cu")
@@
 	)
 	(segment
-		(start 246.289 81.289)
-		(end 246.289 82.595)
+		(start 255.67 50.04)
+		(end 257.0708 48.6392)
 		(width 0.6)
 		(layer "F.Cu")
@@
 	)
 	(segment
-		(start 257.0708 48.6392)
-		(end 257.0708 46.8462)
+		(start 246.57 50.04)
+		(end 255.67 50.04)
 		(width 0.6)
 		(layer "F.Cu")
@@
 	)
 	(segment
-		(start 255.67 50.04)
-		(end 257.0708 48.6392)
+		(start 244 80.75)
+		(end 244 82)
+		(width 0.6)
+		(layer "F.Cu")
+		(net "Net-(IC1-NC)")
+	)
+	(segment
+		(start 257.0708 48.6392)
+		(end 257.0708 46.8462)
 		(width 0.6)
 		(layer "F.Cu")
@@
 	)
 	(via
-		(at 243.24 75.62)
+		(at 243.24 74.5)
 		(size 1)
 		(drill 0.8)
@@
 	)
 	(segment
+		(start 243.24 78.95)
+		(end 243.24 74.5)
+		(width 0.6)
+		(layer "B.Cu")
+		(net "Net-(IC1-NC)")
+	)
+	(segment
 		(start 243.5 79.5)
 		(end 243.5 79.21)
@@
 		(net "Net-(IC1-NC)")
 	)
-	(segment
-		(start 243.24 78.95)
-		(end 243.24 75.62)
-		(width 0.6)
-		(layer "B.Cu")
-		(net "Net-(IC1-NC)")
-	)
-	(segment
-		(start 240.86 83.03)
-		(end 239.32 84.57)
-		(width 0.6)
-		(layer "B.Cu")
-		(net "Net-(U5-Resistance)")
-	)
-	(segment
-		(start 240.86 79.72)
-		(end 240.86 83.03)
-		(width 0.6)
-		(layer "B.Cu")
-		(net "Net-(U5-Resistance)")
-	)
-	(segment
-		(start 239.32 84.57)
-		(end 233.89 84.57)
-		(width 0.6)
-		(layer "B.Cu")
-		(net "Net-(U5-Resistance)")
-	)
-	(segment
-		(start 233.89 84.57)
-		(end 228.46 90)
-		(width 0.6)
-		(layer "B.Cu")
-		(net "Net-(U5-Resistance)")
-	)
 	(zone

Commit message: Ancre_v13_test_DRC
Routing:
- net Net-(IC1-RXD): track 36.9 -> 38.4 mm
Changed lines of the file:
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@@
 	)
 	(segment
-		(start 255.55 76.955)
-		(end 251.595 73)
-		(width 0.6)
-		(layer "B.Cu")
-		(net "Net-(IC1-RXD)")
-	)
-	(segment
-		(start 253.5 82.595)
-		(end 254.515 82.595)
+		(start 255.55 81.56)
+		(end 255.55 76.955)
 		(width 0.6)
 		(layer "B.Cu")
@@
 	(segment
 		(start 251.595 73)
-		(end 233.52 73)
-		(width 0.6)
-		(layer "B.Cu")
-		(net "Net-(IC1-RXD)")
-	)
-	(segment
-		(start 233.52 73)
-		(end 230.42 76.1)
+		(end 231 73)
 		(width 0.6)
 		(layer "B.Cu")
@@
 	)
 	(segment
-		(start 255.55 81.56)
-		(end 255.55 76.955)
+		(start 255.55 76.955)
+		(end 251.595 73)
 		(width 0.6)
 		(layer "B.Cu")
+		(net "Net-(IC1-RXD)")
+	)
+	(segment
+		(start 231 73)
+		(end 230.42 73.58)
+		(width 0.6)
+		(layer "B.Cu")
+		(net "Net-(IC1-RXD)")
+	)
+	(segment
+		(start 230.42 73.58)
+		(end 230.42 76.1)
+		(width 0.6)
+		(layer "B.Cu")
+		(net "Net-(IC1-RXD)")
+	)
+	(segment
+		(start 253.5 82.595)
+		(end 254.515 82.595)
+		(width 0.6)
+		(layer "B.Cu")

Commit message: gbr
Routing:
- net Net-(IC1-RXD): track 38.4 -> 50.4 mm
- net +5V: track 46.3 -> 51.5 mm
- net Net-(IC1-TXD): track 38.5 -> 42.4 mm
Changed lines of the file:
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@@
 		(filling no)
 		(pcbplotparams
-			(layerselection 0x00000000_00000000_55555555_5755f5ff)
-			(plot_on_all_layers_selection 0x00000000_00000000_00000000_00000000)
+			(layerselection 0x00000000_00000000_55555555_57555555)
+			(plot_on_all_layers_selection 0x00000000_00000000_00000000_02000000)
 			(disableapertmacros no)
 			(usegerberextensions no)
@@
 			(outputformat 1)
 			(mirror no)
-			(drillshape 1)
+			(drillshape 0)
 			(scaleselection 1)
 			(outputdirectory "")
@@
 	(via
 		(at 244.365 83.865)
-		(size 1)
+		(size 1.1)
 		(drill 0.8)
 		(layers "F.Cu" "B.Cu")
@@
 	)
 	(segment
+		(start 256.75 74.25)
+		(end 258.02 75.52)
+		(width 0.8)
+		(layer "F.Cu")
+		(net "+5V")
+	)
+	(segment
 		(start 255.32 83.94)
 		(end 255.32 84.2)
@@
 	)
 	(segment
-		(start 240.1 77.51)
-		(end 240.11 77.5)
-		(width 0.8)
-		(layer "F.Cu")
-		(net "+5V")
-	)
-	(segment
-		(start 254.88 77.5)
-		(end 258.02 80.64)
-		(width 0.8)
-		(layer "F.Cu")
-		(net "+5V")
-	)
-	(segment
-		(start 238.69 76.1)
-		(end 235.5 76.1)
+		(start 239.15 76.1)
+		(end 241 74.25)
 		(width 0.8)
 		(layer "F.Cu")
@@
 	)
 	(segment
-		(start 240.1 77.51)
-		(end 238.69 76.1)
+		(start 258.02 75.52)
+		(end 258.02 81.97)
 		(width 0.8)
 		(layer "F.Cu")
@@
 	)
 	(segment
-		(start 239.65 77.51)
-		(end 237.31 79.85)
+		(start 258.02 81.97)
+		(end 257.99 82)
 		(width 0.8)
 		(layer "F.Cu")
@@
 	)
 	(segment
-		(start 258.02 81.97)
-		(end 257.99 82)
+		(start 241 74.25)
+		(end 256.75 74.25)
 		(width 0.8)
 		(layer "F.Cu")
@@
 	)
 	(segment
-		(start 258.02 80.64)
-		(end 258.02 81.97)
+		(start 235.5 78.04)
+		(end 237.31 79.85)
 		(width 0.8)
 		(layer "F.Cu")
@@
 	)
 	(segment
-		(start 240.11 77.5)
-		(end 254.88 77.5)
+		(start 235.5 76.1)
+		(end 235.5 78.04)
 		(width 0.8)
 		(layer "F.Cu")
@@
 	)
 	(segment
-		(start 240.1 77.51)
-		(end 239.65 77.51)
+		(start 235.5 76.1)
+		(end 239.15 76.1)
 		(width 0.8)
 		(layer "F.Cu")
@@
 	)
 	(segment
-		(start 240.67 75.19)
-		(end 240.67 73.4)
+		(start 228.75 71.5)
+		(end 227.88 72.37)
 		(width 0.6)
 		(layer "F.Cu")
@@
 	)
 	(segment
-		(start 249.905 86.405)
-		(end 251.711 86.405)
-		(width 0.6)
-		(layer "F.Cu")
-		(net "Net-(IC1-TXD)")
-	)
-	(segment
-		(start 240.67 73.4)
-		(end 240.39 73.12)
+		(start 249.09 77)
+		(end 249 77.09)
 		(width 0.6)
 		(layer "F.Cu")
@@
 	)
 	(segment
-		(start 227.88 74.04)
-		(end 227.88 76.1)
-		(width 0.6)
-		(layer "F.Cu")
-		(net "Net-(IC1-TXD)")
-	)
-	(segment
-		(start 228.8 73.12)
-		(end 227.88 74.04)
+		(start 249.09 76.5)
+		(end 249.09 77)
 		(width 0.6)
 		(layer "F.Cu")
@@
 	)
 	(segment
-		(start 240.39 73.12)
-		(end 228.8 73.12)
+		(start 249 77.09)
+		(end 249 85.5)
 		(width 0.6)
 		(layer "F.Cu")
@@
 	)
 	(segment
-		(start 241.48 76)
-		(end 240.67 75.19)
+		(start 249 71.5)
+		(end 228.75 71.5)
 		(width 0.6)
 		(layer "F.Cu")
@@
 	)
 	(segment
-		(start 249.09 76)
-		(end 241.48 76)
+		(start 227.88 72.37)
+		(end 227.88 76.1)
 		(width 0.6)
 		(layer "F.Cu")
@@
 	)
 	(segment
-		(start 249 84)
-		(end 249 85.5)
+		(start 249.905 86.405)
+		(end 251.711 86.405)
 		(width 0.6)
 		(layer "F.Cu")
@@
 	)
 	(via
-		(at 249.09 76)
-		(size 1)
+		(at 249 71.5)
+		(size 1.1)
 		(drill 0.8)
 		(layers "F.Cu" "B.Cu")
@@
 	)
 	(via
-		(at 249 84)
-		(size 1)
+		(at 249.09 76.5)
+		(size 1.1)
 		(drill 0.8)
 		(layers "F.Cu" "B.Cu")
@@
 	)
 	(segment
-		(start 249.09 76)
-		(end 249.09 83.91)
+		(start 249 71.5)
+		(end 249 74.5)
 		(width 0.6)
 		(layer "B.Cu")
@@
 	)
 	(segment
-		(start 249.09 83.91)
-		(end 249 84)
+		(start 249 74.5)
+		(end 249.09 74.59)
+		(width 0.6)
+		(layer "B.Cu")
+		(net "Net-(IC1-TXD)")
+	)
+	(segment
+		(start 249.09 74.59)
+		(end 249.09 76.5)
 		(width 0.6)
 		(layer "B.Cu")
@@
 	(via
 		(at 253.5 82.595)
-		(size 1)
+		(size 1.1)
 		(drill 0.8)
 		(layers "F.Cu" "B.Cu")
@@
 	)
 	(segment
-		(start 255.55 81.56)
-		(end 255.55 76.955)
+		(start 255.55 68.8)
+		(end 254.25 67.5)
 		(width 0.6)
 		(layer "B.Cu")
@@
 	)
 	(segment
-		(start 251.595 73)
-		(end 231 73)
+		(start 254.25 67.5)
+		(end 232 67.5)
 		(width 0.6)
 		(layer "B.Cu")
@@
 	)
 	(segment
-		(start 254.515 82.595)
-		(end 255.55 81.56)
+		(start 232 67.5)
+		(end 230.42 69.08)
 		(width 0.6)
 		(layer "B.Cu")
@@
 	)
 	(segment
-		(start 255.55 76.955)
-		(end 251.595 73)
+		(start 253.5 82.595)
+		(end 254.515 82.595)
 		(width 0.6)
 		(layer "B.Cu")
@@
 	)
 	(segment
-		(start 231 73)
-		(end 230.42 73.58)
+		(start 254.515 82.595)
+		(end 255.55 81.56)
 		(width 0.6)
 		(layer "B.Cu")
@@
 	)
 	(segment
-		(start 230.42 73.58)
+		(start 230.42 69.08)
 		(end 230.42 76.1)
 		(width 0.6)
@@
 	)
 	(segment
-		(start 253.5 82.595)
-		(end 254.515 82.595)
+		(start 255.55 81.56)
+		(end 255.55 68.8)
 		(width 0.6)
 		(layer "B.Cu")
@@
 	)
 	(segment
-		(start 243.24 53.37)
-		(end 246.57 50.04)
+		(start 257.0708 48.6392)
+		(end 257.0708 46.8462)
 		(width 0.6)
 		(layer "F.Cu")
@@
 	)
 	(segment
-		(start 244 82)
-		(end 244.595 82.595)
+		(start 243.24 53.37)
+		(end 246.57 50.04)
 		(width 0.6)
 		(layer "F.Cu")
@@
 	)
 	(segment
-		(start 243.24 74.5)
-		(end 243.24 53.37)
+		(start 246.57 50.04)
+		(end 255.67 50.04)
 		(width 0.6)
 		(layer "F.Cu")
@@
 	)
 	(segment
-		(start 244 80)
-		(end 243.5 79.5)
+		(start 244 82)
+		(end 244.595 82.595)
 		(width 0.6)
 		(layer "F.Cu")
@@
 	)
 	(segment
-		(start 255.67 50.04)
-		(end 257.0708 48.6392)
+		(start 244 80)
+		(end 243.5 79.5)
 		(width 0.6)
 		(layer "F.Cu")
@@
 	)
 	(segment
-		(start 246.57 50.04)
-		(end 255.67 50.04)
+		(start 255.67 50.04)
+		(end 257.0708 48.6392)
 		(width 0.6)
 		(layer "F.Cu")
@@
 	)
 	(segment
-		(start 257.0708 48.6392)
-		(end 257.0708 46.8462)
+		(start 243.24 70)
+		(end 243.24 53.37)
 		(width 0.6)
 		(layer "F.Cu")
@@
 	(via
 		(at 243.5 79.5)
-		(size 1)
+		(size 1.1)
 		(drill 0.8)
 		(layers "F.Cu" "B.Cu")
@@
 	)
 	(via
-		(at 243.24 74.5)
-		(size 1)
+		(at 243.24 70)
+		(size 1.1)
 		(drill 0.8)
 		(layers "F.Cu" "B.Cu")
@@
 	)
 	(segment
-		(start 243.24 78.95)
-		(end 243.24 74.5)
-		(width 0.6)
-		(layer "B.Cu")
-		(net "Net-(IC1-NC)")
-	)
-	(segment
 		(start 243.5 79.5)
 		(end 243.5 79.21)
@@
 		(layer "B.Cu")
 		(net "Net-(IC1-NC)")
+	)
+	(segment
+		(start 243.24 78.95)
+		(end 243.24 70)
+		(width 0.6)
+		(layer "B.Cu")
+		(net "Net-(IC1-NC)")
